Commit message: last

File: roscue_arm_description/urdf/assemblies/roscue_arm.urdf.xacro (robot description, xacro)
@@ -142,5 +142,5 @@
       <origin xyz="-0.065000 0.000000 0.063000" rpy="0.000000 -1.570796 0.000000"/>
       <axis xyz="-0.000000 -0.000000 -1.000000"/>
-      <limit lower="-1.5708" upper="1.5708" effort="100.0" velocity="1.00"/>
+      <limit lower="-1.4835" upper="1.5708" effort="100.0" velocity="1.00"/>
     </joint>
     <joint name="${prefix}arm_joint_2" type="revolute">
@@ -149,5 +149,5 @@
       <origin xyz="0.340500 0.000000 0.058500" rpy="-1.570796 -0.000000 -1.570796"/>
       <axis xyz="0.000000 1.000000 0.000000"/>
-      <limit lower="-1.3963" upper="1.3963" effort="100.0" velocity="1.00"/>
+      <limit lower="-1.3631" upper="1.3963" effort="100.0" velocity="1.00"/>
     </joint>
     <joint name="${prefix}arm_joint_3" type="revolute">
@@ -156,5 +156,5 @@
       <origin xyz="-0.000500 0.019500 0.180000" rpy="-0.000000 0.000000 0.000000"/>
       <axis xyz="0.000000 1.000000 0.000000"/>
-      <limit lower="-1.5708" upper="1.5708" effort="100.0" velocity="1.00"/>
+      <limit lower="-1.5970" upper="1.5708" effort="100.0" velocity="1.00"/>
     </joint>
     <joint name="${prefix}arm_joint_4" type="revolute">
@@ -163,5 +163,5 @@
       <origin xyz="-0.000000 0.002500 0.090000" rpy="0.000000 -0.000000 1.570796"/>
       <axis xyz="-0.000000 0.000000 1.000000"/>
-      <limit lower="-2.9671" upper="2.9671" effort="100.0" velocity="1.00"/>
+      <limit lower="-1.5708" upper="1.5708" effort="100.0" velocity="1.00"/>
     </joint>
     <!-- ROS 2 control: generated generic system -->

File: roscue_arm_description/urdf/roscue_arm.urdf.xacro (robot description, xacro)
@@ -97,10 +97,10 @@
     <limit lower="-1.9426" upper="1.9426" effort="100.0" velocity="1.00"/>
   </joint>
-  <!-- ROS 2 control: generated generic system -->
-  <ros2_control name="roscue_arm_system" type="system">
+  <!-- ROS 2 control: gripper-only mock system. -->
+  <ros2_control name="roscue_gripper_system" type="system">
     <hardware>
       <plugin>mock_components/GenericSystem</plugin>
-      <param name="cmd_topic">sim/roscue_arm_system/cmd</param>
-      <param name="state_topic">sim/roscue_arm_system/state</param>
+      <param name="cmd_topic">sim/roscue_gripper_system/cmd</param>
+      <param name="state_topic">sim/roscue_gripper_system/state</param>
     </hardware>
     <joint name="finger_1_base_joint">
@@ -186,3 +186,30 @@
     </joint>
   </ros2_control>
+  <!--
+    RealSense wrist mount. The camera driver owns camera_link's optical-frame
+    children; robot_state_publisher only connects the camera to the arm.
+    Replace this provisional transform after measuring the physical mount.
+  -->
+  <link name="camera_link">
+    <visual>
+      <origin xyz="0 0 0" rpy="0 0 0"/>
+      <geometry>
+        <box size="0.090 0.025 0.025"/>
+      </geometry>
+      <material name="camera_gray">
+        <color rgba="0.2 0.2 0.2 1.0"/>
+      </material>
+    </visual>
+    <collision>
+      <origin xyz="0 0 0" rpy="0 0 0"/>
+      <geometry>
+        <box size="0.090 0.025 0.025"/>
+      </geometry>
+    </collision>
+  </link>
+  <joint name="camera_mount_joint" type="fixed">
+    <parent link="gripper_base_link"/>
+    <child link="camera_link"/>
+    <origin xyz="0.0 0.0 0.07" rpy="0.0 0.0 0.0"/>
+  </joint>
 </robot>
